File: 4in1ESC-30x30.kicad_sch (KiCad schematic)
At the start: 62 parts, among them J1 SM08B-SRSS-TB, U1 INA199A1DCKR, U18 LMR51420YDDCR, U26 TPS746-3.3DRV, U5 XRIM160808SR47MBCD

Commit message: Sync v0.4 component changes from 20x20 variant
- INA186A3IDCKR replaces INA199A1DCKR (current sense amp)
- TLV76733DRVR replaces TPS746 (LDO), SNS wired to output
- BLM03PX121SN1D ferrite bead on VDDA
- Add .gitignore for backups and prl files

Co-Authored-By: Claude Opus 4.6 <noreply@anthropic.com>
Parts:
- removed C30, C52, C54, C55, C56, C58, C60, C61, C62: 10uF, Capacitor_SMD:C_0805_2012Metric, symbol Device:C
- removed J1: SM08B-SRSS-TB, Connector_JST:JST_SH_SM08B-SRSS-TB_1x08-1MP_P1.00mm_Horizontal, symbol SM08B-SRSS-TB:SM08B-SRSS-TB
- removed U1: INA199A1DCKR, Package_TO_SOT_SMD:SOT-363_SC-70-6, symbol Amplifier_Current:INA199xxDCK
- removed U26: TPS746-3.3DRV, Package_SON:WSON-6-1EP_2x2mm_P0.65mm_EP1x1.6mm, symbol Regulator_Linear:LP5912-3.3DRV
- added J1: SM08B-SRSS-TB, 4in1ESC-30x30:JST_SM08B-SRSS-TB, symbol components:SM08B-SRSS-TB
- added U1: TLV76733DRVR, 4in1ESC-30x30:WSON-6_L2.0-W2.0-P0.65-TL-EP, symbol components:TLV76733DRVR
- added U12: INA186A3IDCKR, 4in1ESC-30x30:SOT-363_SC-70-6, symbol components:INA186A3IDCKR
- U18: LCSC C5383002 -> C7296200
Connections:
- net +3V3: now also U1.2 (FB/SNS), U12.3 (VS)
- net +8V: now also U1.4 (EN), U1.6 (IN)
- net +BATT: now also J1.1, U12.5 (-IN)
- net CURR: now also J1.3
- net GND: now also J1.2, J1.P1 (MP1), J1.P2 (MP2), U1.1 (OUT), U1.3 (GND), U1.5 (GND), U1.7 (EP), U12.1 (REF), U12.2 (GND)
- net M1: now also J1.5
- net M2: now also J1.6
- net M3: now also J1.7
- net M4: now also J1.8
- net at R73.2: now also U12.6 (OUT)
- net CSA+: now reaches Rsense1.1, U4.1 (VBAT)
- net CSA+: now also U12.4 (+IN)
Other:
- note added: "0.2mΩ shunt × 100V/V gain Max: 165A (3.3V ADC)"
- moved on the sheet: C1, C42, C70, C71, C93, C94, R73

Commit message: Prepare for open source: PCB layout, new footprints, 3D models, comprehensive gitignore
- Add PCB layout (4-layer, 30x30mm)
- Add SP40N01GHNK MOSFET footprint and 3D model (PDFN-8L 5x6mm)
- Add NSG20652Q gate driver alt footprint and QFN-24 3D model
- Add board outline footprint and SMB connector footprint/3D model
- Update schematic and symbols for NSG20652Q pinout
- Comprehensive .gitignore matching 20x20 variant
- Fix README link to 20x20 repo

Co-Authored-By: Claude Opus 4.6 <noreply@anthropic.com>
Parts:
- removed C10, C11, C12, C13, C14, C15, C16, C17, C18, C19, C20, C21, C22, C23, C24, C25, C26, C27, C28, C29, C31, C4, C40, C41, C47, C5, C51, C7, C8, C9: 10uF, Capacitor_SMD:C_0805_2012Metric, symbol Device:C
- removed C86: 22uF, Capacitor_SMD:C_0603_1608Metric, symbol Device:C
- removed U4: ~, 4in1ESC-30x30:4in1ESC, symbol Connector:4in1ESC
- added D1: SMBJ26A_C908802, 4in1ESC-30x30:SMB_L4.5-W3.7-LS5.4-RD, symbol components:SMBJ26A_C908802
- added U3: ~, 4in1ESC-30x30:4in1ESC30x30, symbol components:4in1ESC
- C2, C3, C6: footprint Capacitor_SMD:C_0805_2012Metric -> Capacitor_SMD:C_1206_3216Metric
- C69, C70, C71, C72, C93, C94: symbol ESCLibrary:GRM033R61C104KE84D -> components:GRM033R61C104KE84D
- R73: symbol ESCLibrary:0201_1kR -> components:0201_1kR
- U18: footprint components:SOT-23-6_L2.9-W1.6-P0.95-LS2.9-BL -> 4in1ESC-30x30:SOT-23-6_L2.9-W1.6-P0.95-LS2.9-BL
- U5: footprint components:IND-SMD_L1.6-W0.8_FTC160865SR47MBCA -> 4in1ESC-30x30:IND-SMD_L1.6-W0.8_FTC160865SR47MBCA
Connections:
- net +3V3: now also U1.1 (OUT)
- net +BATT: now also D1.1, U3.3 (VBAT+)
- net CSA+: now also U3.1 (VBAT)
- net CURR: now also U3.5 (CUR)
- net ESC1/A: now also U3.23 (1A)
- net ESC1/B: now also U3.22 (1B)
- net ESC1/C: now also U3.21 (1C)
- net ESC2/A: now also U3.20 (2B)
- net ESC2/B: now also U3.19 (2C)
- net ESC2/C: now also U3.18 (2A)
- net ESC3/A: now also U3.15 (3B)
- net ESC3/B: now also U3.16 (3C)
- net ESC3/C: now also U3.17 (3A)
- net ESC4/A: now also U3.12 (4A)
- net ESC4/B: now also U3.13 (4B)
- net ESC4/C: now also U3.14 (4C)
- net GND: now also D1.2, U3.11 (Hole), U3.2 (BATGND), U3.4 (GND); no longer U1.1 (OUT)
- net M1: now also U3.7 (M1)
- net M2: now also U3.8 (M2)
- net M3: now also U3.9 (M3)
- net M4: now also U3.10 (M4)
