File: 4in1ESC-30x30.kicad_sch (KiCad schematic)
At the start: 23 parts, among them J1 SM08B-SRSS-TB, U1 TLV76733DRVR, U12 INA186A3IDCKR, U18 LMR51420YDDCR, U5 XRIM160808SR47MBCD

Commit message: Final parts changes and production files for V0.1
Parts:
- C2, C3, C6: LCSC C440198 -> C13585
- D1: LCSC Part C908802 -> C123820
