File: 4in1ESC-30x30.kicad_sch (KiCad schematic)
At the start: 23 parts, among them J1 SM08B-SRSS-TB, U1 TLV76733DRVR, U12 INA186A3IDCKR, U18 LMR51420YDDCR, U5 XRIM160808SR47MBCD

Commit message: Replace backordered parts with in-stock LCSC alternatives
- 10kΩ 0201: C473048 → C106225 (Yageo, 662k stock)
- Ferrite bead 0201: C525479 → C440127 (330Ω@100MHz, better for VDDA filtering)
- 220Ω 0201: C473535 → C226468 (Yageo)
- 10uF cap: C440198 (0805) → C13585 (1206 basic part, Samsung)
- TVS diode: C908802 → C315992 (Littelfuse SMBJ26A)

Co-Authored-By: Claude Opus 4.6 (1M context) <noreply@anthropic.com>
Parts:
- D1: LCSC Part C123820 -> C315992
- R118: LCSC C473048 -> C106225
- U3: now left out of the parts list

Commit message: Standardize repo: .gitignore, README, license, remove production from tracking
- Standardize .gitignore to match ecosystem template
- Update README: simplify license section, remove stale status checklist
- Replace LICENSE stub with full CERN-OHL-S-2.0 text
- Remove production/ from git tracking (generated, re-exportable)
- Add previously untracked licensing/ directory
- Delete empty nextpcb/ directory

Co-Authored-By: Claude Opus 4.6 (1M context) <noreply@anthropic.com>
Parts:
- C2, C3, C6: LCSC C13585 -> C89632
Changed lines of the file:
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@@
 			)
 		)
-		(property "LCSC" "C13585"
+		(property "LCSC" "C89632"
 			(at 78.74 67.31 0)
 			(effects
@@
 			)
 		)
-		(property "LCSC" "C13585"
+		(property "LCSC" "C89632"
 			(at 64.77 67.31 0)
 			(effects
@@
 			)
 		)
-		(property "LCSC" "C13585"
+		(property "LCSC" "C89632"
 			(at 92.71 67.31 0)
 			(effects
