File: 4in1ESC-30x30.kicad_sch (KiCad schematic)
At the start: 23 parts, among them J1 SM08B-SRSS-TB, U1 TLV76733DRVR, U12 INA186A3IDCKR, U18 LMR51420YDDCR, U5 XRIM160808SR47MBCD

Commit message: alpha routing
Parts:
- removed C1, C42: 22uF, Capacitor_SMD:C_0402_1005Metric, symbol Device:C
- removed C43: 22uF, Capacitor_SMD:C_0603_1608Metric, symbol Device:C
- removed C69, C70, C71, C72: 100nF, Capacitor_SMD:C_0201_0603Metric, symbol components:GRM033R61C104KE84D
- removed R118: 10k, Capacitor_SMD:C_0201_0603Metric, symbol Device:R
- removed R119: 124k, Resistor_SMD:R_0201_0603Metric, symbol Device:R
- removed U1: TLV76733DRVR, 4in1ESC-30x30:WSON-6_L2.0-W2.0-P0.65-TL-EP, symbol components:TLV76733DRVR
- removed U18: LMR51420YDDCR, 4in1ESC-30x30:SOT-23-6_L2.9-W1.6-P0.95-LS2.9-BL, symbol components:LMR51420YDDCR
- removed U5: XRIM160808SR47MBCD, 4in1ESC-30x30:IND-SMD_L1.6-W0.8_FTC160865SR47MBCA, symbol components:XRIM160808SR47MBCD
- added C4, C51: 22uF, Capacitor_SMD:C_0402_1005Metric, symbol Device:C
- added C47, C86: 22uF, Capacitor_SMD:C_0603_1608Metric, symbol Device:C
- added C74, C75, C76, C81: 100nF, Capacitor_SMD:C_0201_0603Metric, symbol ESCLibrary:GRM033R61C104KE84D
- added D2, D3: SMBJ24A, 4in1ESC-30x30:SMB_L4.5-W3.7-LS5.4-RD, symbol components:SMBJ26A_C908802
- added R120: 115k, Resistor_SMD:R_0201_0603Metric, symbol Device:R
- added R121: 10k, 4in1ESC:R_0201_0603Metric, symbol Device:R
- added Rsense2: 0.2mR, Resistor_SMD:R_2512_6332Metric, symbol Device:R
- added U13: LMR54406DBVR, 4in1ESC:SOT-23-6_L2.9-W1.6-P0.95-LS2.8-BR, symbol components:LMR54406DBVR
- added U14: FTC160808S4R7MBCA, 4in1ESC:IND-SMD_L1.6-W0.8_FTC160865SR47MBCA, symbol components:XRIM160808SR47MBCD
- added U15: TLV76733DRVR, 4in1ESC:WSON-6_L2.0-W2.0-P0.65-TL-EP, symbol components:TLV76733DRVR
- D1: value SMBJ26A_C908802 -> SMBJ24A; LCSC Part C315992 -> C19077578
- U3: value ~ -> (none)
Connections:
- net +3V3: now also C4.2, C51.2, C81.1, U15.1 (OUT), U15.2 (FB/SNS)
- net +BATT: now also C74.1, D2.1, D3.1, Rsense2.2, U13.4 (EN), U13.5 (VIN)
- net CSA+: now also Rsense2.1
- net GND: now also C4.1, C47.2, C51.1, C74.2, C76.2, C81.2, C86.2, D2.2, D3.2, R121.2, U13.2 (GND), U15.3 (GND), U15.5 (GND), U15.7 (EP)
- new net: R120.2, R121.1, U13.3 (FB)
- new net: C75.1, U13.6 (SW), U14.1
- new net: C75.2, U13.1 (CB)
- new net +10V: C47.1, C76.1, C86.1, R120.1, U14.2, U15.4 (EN), U15.6 (IN)
