File: ESC.kicad_sch (KiCad schematic)
At the start: 36 parts, among them Q1 C22385416, Q11 C22385416, Q16 C22385416, Q2 C22385416, Q21 C22385416, Q6 C22385416, U2 AT32F421G8U7, U4 NSG2065Q

Commit message: alpha routing
Parts:
- removed C32, C36, C53: 100nF, Capacitor_SMD:C_0402_1005Metric, symbol components:GRM033R61C104KE84D
- removed C48, C49, C50, C57: 100nF, Capacitor_SMD:C_0201_0603Metric, symbol components:GRM033R61C104KE84D
- removed FB2: BLM03PX121SN1D, Inductor_SMD:L_0201_0603Metric, symbol Device:FerriteBead_Small
- removed R16, R2, R43, R60, R9: 8R, Capacitor_SMD:C_0201_0603Metric, symbol PCM_Resistor_AKL:R_0402
- removed R18, R19: 10k, Capacitor_SMD:C_0201_0603Metric, symbol components:0201_10kR
- removed R20: 220R, Resistor_SMD:R_0201_0603Metric, symbol components:0201_220R
- removed U2: AT32F421G8U7, 4in1ESC-30x30:QFN-28_L4.0-W4.0-P0.40-TL-EP2.4, symbol components:AT32F421G8U7
- added C32, C36, C53: 100nF, Capacitor_SMD:C_0402_WIDE, symbol ESCLibrary:GRM033R61C104KE84D
- added C48, C49, C50, C57: 100nF, Capacitor_SMD:C_0201_0603Metric, symbol ESCLibrary:GRM033R61C104KE84D
- added R18, R19: 10k, Resistor_SMD:R_0201_0603Metric, symbol ESCLibrary:0201_10kR
- added R20: 220R, Resistor_SMD:R_0201_0603Metric, symbol ESCLibrary:0201_220R
- added R42, R55, R62, R76, R80: 15R, Resistor_SMD:R_0201_0603Metric, symbol PCM_Resistor_AKL:R_0402
- added R84: 10R, Resistor_SMD:R_0201_0603Metric, symbol Device:R
- added U2: AT32F421G8U7, 4in1ESC:QFN-28_L4.0-W4.0-P0.40-TL-EP2.4, symbol ESCLibrary:AT32F421G8U7
- R23: value 8R -> 15R; footprint Capacitor_SMD:C_0201_0603Metric -> Resistor_SMD:R_0201_0603Metric
- U4: footprint 4in1ESC-30x30:QFN-24_L4.0-W4.0-P0.50-TL-EP2.8 -> 4in1ESC:QFN-24_L4.0-W4.0-P0.50-TL-EP2.8
Connections:
- net +3V3: now also C49.1, R18.2, R84.2, U2.17 (VDD)
- net A: now also C53.1
- net AH: now also U2.20 (PA10)
- net AL: now also U2.15 (PB1)
- net B: now also C32.1
- net BH: now also U2.19 (PA9)
- net BL: now also U2.14 (PB0)
- net C: now also C36.1
- net CH: now also U2.18 (PA8)
- net CL: now also U2.13 (PA7)
- net FBA: now also U2.6 (PA0)
- net FBB: now also U2.10 (PA4)
- net FBC: now also U2.11 (PA5)
- net FBCOMMON: now also U2.7 (PA1)
- net GHA: now also R76.1
- net GHB: now also R55.1
- net GHC: now also R23.1
- net GLA: now also R80.1
- net GLB: now also R62.1; no longer R23.1
- net GLC: now also R42.1
- net GND: now also C48.2, C49.2, C50.2, C57.2, R19.2, U2.16 (VSS), U2.29 (VSS)
- net dshot: now also R20.1
- net at Q6.2 (G): now also R55.2
- net at TP1.1: now also U2.21 (PA13)
- net at Q11.2 (G): now also R62.2; no longer R23.2
- net at Q2.2 (G): now also R80.2
- net at Q1.2 (G): now also R76.2
- net at U4.17 (VB2): now also C32.2
- net at Q16.2 (G): now also R23.2
- net at U4.20 (VB1): now also C53.2
- net at Q21.2 (G): now also R42.2
- net at TP4.1: now also U2.22 (PA14)
- net at U4.14 (VB3): now also C36.2
- net +8V renamed +10V
- net +10V: now also C57.1
- new net: R20.2, U2.25 (PB4)
- new net: R19.1, U2.1 (BOOT0)
- new net: C50.1, R18.1, U2.4 (NRST)
- new net vdda: C48.1, R84.1, U2.5 (VDDA)
Other:
- note added: "XRS280N03C selected (C50314140, 30V/280A/0.5mÎ©, PDFN-8L 5Ã6, drop-in footprint)"
