File: ESC.kicad_sch (KiCad schematic)
At the start: 36 parts, among them Q1 C22385416, Q11 C22385416, Q16 C22385416, Q2 C22385416, Q21 C22385416, Q6 C22385416, U2 AT32F421G8U7, U4 NSG2065Q

Commit message: meta: standardize symbol BOM/doc fields (30x30)
Add MPN/Manufacturer/LCSC/Digi-Key/Mouser/Farnell/Cost to every sourced
part. Source MPN + LCSC unit cost via keyless LCSC; Manufacturer set for
known ICs (TI, ArteryTek, Littelfuse). Fix MOSFET Value/LCSC swap
(Value/MPN=SP40N01GHNK, LCSC=C22385416), clear legacy LCSC_Part, strip
CJK from Manufacturer. Digi-Key/Mouser/Farnell left blank pending API
creds. Properties-only — no connectivity change. Also carries the
finalized on-canvas design comments.

Co-Authored-By: Claude Opus 4.8 (1M context) <noreply@anthropic.com>
Parts:
- C32, C36, C53: Cost (none) -> 0.003257; MPN (none) -> CL05B104KB54PNC
- C48, C49, C50, C57: Cost (none) -> 0.008457; MPN (none) -> GRM033R6YA104KE14D
- Q1, Q11, Q16, Q2, Q21, Q6: value C22385416 -> SP40N01GHNK; Cost (none) -> 0.3843; LCSC SP40N01GHNK -> C22385416; MPN (none) -> SP40N01GHNK
- R18, R19, R25, R27, R28, R30, R31, R33: Cost (none) -> 0.0007714; MPN (none) -> RC0201FR-0710KL
- R20: Cost (none) -> 0.001529; MPN (none) -> AC0201FR-07220RL
- R23, R42, R55, R62, R76, R80: Cost (none) -> 0.0006286; MPN (none) -> 0201WMF150JTEE
- R26, R29, R32: Cost (none) -> 0.0006; MPN (none) -> 0201WMF1001TEE
- R84: Cost (none) -> 0.0017; MPN (none) -> RC0201FR-0710RL
- U2: Cost (none) -> 0.76; MPN (none) -> AT32F421G8U7; Manufacturer (none) -> ArteryTek
- U4: Cost (none) -> 0.3657; MPN (none) -> NSG2065Q
Other:
- note added: "(gate driver has integrated diode)"
- note added: "06/06/2026"
- note added: "2"
- note added: "BEMF Feedback network"
- note added: "Bootstrap capacitors for high side N-MOS switching"
- note added: "Gate Driver"
- note added: "LPF on VDDA"
- note added: "MOSFET, low and high side for each phase"
- note added: "Microcontroller: AT32"
- note added: "SWC flashing"
- note added: "Single sheet instance of an ESC, duplicated 4 times"
