File: 4in1.kicad_sch (KiCad schematic)
At the start: 27 parts, among them J1 SM08B-SRSS-TB, U12 INA186A3IDCKR, U13 LMR54406DBVR, U14 FTC160808S4R7MBCA, U15 TLV76733DRVR

Commit message: meta: standardize symbol BOM/doc fields (30x30)
Add MPN/Manufacturer/LCSC/Digi-Key/Mouser/Farnell/Cost to every sourced
part. Source MPN + LCSC unit cost via keyless LCSC; Manufacturer set for
known ICs (TI, ArteryTek, Littelfuse). Fix MOSFET Value/LCSC swap
(Value/MPN=SP40N01GHNK, LCSC=C22385416), clear legacy LCSC_Part, strip
CJK from Manufacturer. Digi-Key/Mouser/Farnell left blank pending API
creds. Properties-only — no connectivity change. Also carries the
finalized on-canvas design comments.

Co-Authored-By: Claude Opus 4.8 (1M context) <noreply@anthropic.com>
Parts:
- C2, C3, C6: Cost (none) -> 0.05129; MPN (none) -> CL31B106KBHNNNE
- C4, C51: Cost (none) -> 0.037; MPN (none) -> CL05A226MQ5QUNC
- C47, C86: Cost (none) -> 0.04157; MPN (none) -> CL10A226MO7JZNC
- C74, C75, C76, C81, C93, C94: Cost (none) -> 0.008457; MPN (none) -> GRM033R6YA104KE14D
- D1, D2, D3: Cost (none) -> 0.04457; LCSC (none) -> C19077578; MPN (none) -> SMBJ24A
- J1: Cost (none) -> 0.2523; MPN (none) -> SM08B-SRSS-TB(LF)(SN)
- R120: Cost (none) -> 0.0005429; MPN (none) -> RTT011153FTH
- R121: Cost (none) -> 0.0007714; MPN (none) -> RC0201FR-0710KL
- R73: Cost (none) -> 0.0006; MPN (none) -> 0201WMF1001TEE
- Rsense1, Rsense2: Cost (none) -> 0.2657; MPN (none) -> ASR-S-3-0.2F
- U12: Cost (none) -> 0.79; MPN (none) -> INA186A3IDCKR; Manufacturer (none) -> Texas Instruments
- U13: Cost (none) -> 0.4229; LCSC (none) -> C5219316; Manufacturer TI(德州仪器) -> Texas Instruments
- U14: Cost (none) -> 0.1079; MPN (none) -> FTC160808S4R7MBCA
- U15: Cost (none) -> 0.242; MPN (none) -> TLV76733DRVR; Manufacturer (none) -> Texas Instruments
Other:
- note added: "06/06/2026"
- note added: "2"
- note added: "4 to 36V, can handle 50V spikes. TBD on 8S 1.1Mhz, 0.6A (plenty for gate driving)"
- note added: "No telemetry signal pin, handled by Extended DSHOT protocol"
- note added: "Overview of OpenESC"
- note added: "SMBJ24A means there will be some leakage at fully charged 6S (25.2V) but voltage clamping gets improved too, will monitor this tradeoff"
- note added: "Total array of 8x6+2 = 50 decoupling caps At 25V DC Bias, only 1.5uF - 2uF derated per cap, so 75 - 100uF but ver low ESR"
- note added: "two parallel shunts = 0.1 mΩ → 10 mV/A → ~330 A"
- note removed: "0.2mΩ shunt × 100V/V gain Max: 165A (3.3V ADC)"
- moved on the sheet: C4, C47, C51, C74, C75, C76, C81, C86, R120, R121, U13, U15
